Commit message: added minimum Unity support with correct vacuum_gripper IK

File: src/kuka_kr10_support/urdf/kr10r1420.urdf (robot description, URDF)
Before this commit: robot kuka_kr10r1420, 11 links, 10 joints
Links:
- added link gripper_tip
- link vacuum_gripper: geometry collision box size=0.1 0.1 0.20; visual box size=0.1 0.1 0.20
Joints:
- added joint gripper_tip_joint: type fixed, parent vacuum_gripper, child gripper_tip, origin xyz=0 0 0.20 rpy=0 0 0

File: src/kuka_kr10_support/urdf/kr10r1420_macro.xacro (robot description, xacro)
@@ -172,9 +172,11 @@
     </joint>
     <!-- I INSERTED VACUUM GRIPPER HERE -->
+    <!-- VACUUM GRIPPER START -->
     <link name="${prefix}vacuum_gripper">
       <visual>
-        <origin xyz="0 0 0.10" rpy="0 0 0"/>  <!-- Центр бокса на полпути вверх -->
-        <geometry>
-          <box size="0.1 0.1 0.2"/>
+        <!-- Центр смещен к основанию (началу) гриппера -->
+        <origin xyz="0 0 0.10" rpy="0 0 0"/>  <!-- Смещение на половину длины -->
+        <geometry>
+          <box size="0.1 0.1 0.20"/>  <!-- Длина 0.20 м по Z -->
         </geometry>
         <material name="grey">
@@ -185,14 +187,23 @@
         <origin xyz="0 0 0.10" rpy="0 0 0"/>
         <geometry>
-          <box size="0.1 0.1 0.2"/>
-        </geometry>
-      </collision>
-    </link>
+          <box size="0.1 0.1 0.20"/>
+        </geometry>
+      </collision>
+    </link>
+    <!-- VACUUM GRIPPER END -->
     <joint name="${prefix}tool0-vacuum_gripper" type="fixed">
       <parent link="${prefix}tool0"/>
       <child link="${prefix}vacuum_gripper"/>
+      <!-- Нулевое смещение - гриппер начинается сразу от tool0 -->
       <origin xyz="0 0 0" rpy="0 0 0"/>
     </joint>
-    <!-- VACUUM GRIPPER END-->
+        <!-- Фрейм на КОНЧИКЕ гриппера -->
+    <link name="${prefix}gripper_tip"/>
+    <joint name="${prefix}gripper_tip_joint" type="fixed">
+      <parent link="${prefix}vacuum_gripper"/>
+      <child link="${prefix}gripper_tip"/>
+      <!-- Смещение на полную длину гриппера (0.20 м) -->
+      <origin xyz="0 0 0.20" rpy="0 0 0"/>
+    </joint>
   </xacro:macro>
 </robot>
